File: hev-controller 1.1.sch (EAGLE design)
At the start: 57 parts, among them CN1 MiniB USB, IC1 ATMEGA32U4-AU, IC2 7805TV, IC3 MCP4822SN, J1 AVR_SPI_PRG_6PTH, U1 MAX232SOIC16, X3 16MHz

Commit message: Upgrade to 1.1
Parts:
- removed EXTPWR: 3PH, SparkFun:M023.5MM
- added JP1: (no value), SparkFun-Connectors:M04PTH
- added Q1: MOSFET-PCHANNELSMD, SparkFun-DiscreteSemi:MOSFET-PCHANNELSMD
Connections:
- new net N$14: C13.+, IC2.VI, Q1.S
- net BLUE-P2: now also BLUETOOTH.4; no longer BLUETOOTH.2
- net BLUE-RX: now also JP1.3, U1.R2OUT; no longer U1.R1OUT
- net BLUE-TX: now also JP1.4, U1.T2IN; no longer U1.T1IN
- net GND: now also BLUETOOTH.1, JP1.2, MEGASQUIRT.1, Q1.G; no longer BLUETOOTH.5, EXTPWR.1, MEGASQUIRT.5
- net SQUIRT-P2: now also MEGASQUIRT.4; no longer MEGASQUIRT.2
- net SQUIRT-RX: now also U1.R1OUT; no longer U1.R2OUT
- net SQUIRT-TX: now also U1.T1IN; no longer U1.T2IN
- net VCC: now also BLUETOOTH.6, JP1.1, MEGASQUIRT.6; no longer BLUETOOTH.9, EXTPWR.2, MEGASQUIRT.9
- net VIN: now also Q1.D; no longer C13.+, IC2.VI
Other:
- note added: "2"
- note removed: "0"
- moved on the sheet: C13
